Commit message: Adding the camera to Robot Chasis + Some Fancy changes

File: urdf/robot.xacro (robot description, xacro)
@@ -1,4 +1,5 @@
 <?xml version='1.0'?>
-<robot name="robot" xmlns:xacro="http://www.ros.org/wiki/xacro">
+<robot name="SHARP_Robot" xmlns:xacro="http://www.ros.org/wiki/xacro">
+_
   <xacro:property name="camera_width" value="0.02"/>
   <xacro:property name="camera_length" value="0.02"/>
@@ -9,5 +10,6 @@
   <xacro:property name="chassis_height" value="0.05"/>
   <xacro:property name="chassis_mass" value="0.5"/>
-  <xacro:property name="wheel_radius" value="0.04"/>
+  <xacro:property name="wheel_radius_front" value="0.04"/>
+  <xacro:property name="wheel_radius_back" value="0.04"/>
   <xacro:property name="wheel_width" value="0.03"/>
   <xacro:property name="wheel_mass" value="0.025"/>
@@ -32,9 +34,9 @@
   </link>
   <link name='wheel_FR'>
-    <xacro:cylinder_inertial name="wheel_FR" m="${wheel_mass}" r="${wheel_radius}" h="${wheel_width}"/>
+    <xacro:cylinder_inertial name="wheel_FR" m="${wheel_mass}" r="${wheel_radius_front}" h="${wheel_width}"/>
     <collision name='wheel_FR_collision'>
       <origin xyz="0 0 0" rpy="1.5708 0 0"/>
       <geometry>
-        <cylinder radius="${wheel_radius}" length="${wheel_width}"/>
+        <cylinder radius="${wheel_radius_front}" length="${wheel_width}"/>
       </geometry>
     </collision>
@@ -42,14 +44,14 @@
       <origin xyz="0 0 0" rpy="1.5708 0 0"/>
       <geometry>
-        <cylinder radius="${wheel_radius}" length="${wheel_width}"/>
+        <cylinder radius="${wheel_radius_front}" length="${wheel_width}"/>
       </geometry>
     </visual>
   </link>
   <link name='wheel_FL'>
-    <xacro:cylinder_inertial name="wheel_FL" m="${wheel_mass}" r="${wheel_radius}" h="${wheel_width}"/>
+    <xacro:cylinder_inertial name="wheel_FL" m="${wheel_mass}" r="${wheel_radius_front}" h="${wheel_width}"/>
     <collision name='wheel_FL_collision'>
       <origin xyz="0 0 0" rpy="1.5708 0 0"/>
       <geometry>
-        <cylinder radius="${wheel_radius}" length="${wheel_width}"/>
+        <cylinder radius="${wheel_radius_front}" length="${wheel_width}"/>
       </geometry>
     </collision>
@@ -57,14 +59,14 @@
       <origin xyz="0 0 0" rpy="1.5708 0 0"/>
       <geometry>
-        <cylinder radius="${wheel_radius}" length="${wheel_width}"/>
+        <cylinder radius="${wheel_radius_front}" length="${wheel_width}"/>
       </geometry>
     </visual>
   </link>
   <link name='wheel_RR'>
-    <xacro:cylinder_inertial name="wheel_RR" m="${wheel_mass}" r="${wheel_radius}" h="${wheel_width}"/>
+    <xacro:cylinder_inertial name="wheel_RR" m="${wheel_mass}" r="${wheel_radius_back}" h="${wheel_width}"/>
     <collision name='wheel_RR_collision'>
       <origin xyz="0 0 0" rpy="1.5708 0 0"/>
       <geometry>
-        <cylinder radius="${wheel_radius}" length="${wheel_width}"/>
+        <cylinder radius="${wheel_radius_back}" length="${wheel_width}"/>
       </geometry>
     </collision>
@@ -72,14 +74,14 @@
       <origin xyz="0 0 0" rpy="1.5708 0 0"/>
       <geometry>
-        <cylinder radius="${wheel_radius}" length="${wheel_width}"/>
+        <cylinder radius="${wheel_radius_back}" length="${wheel_width}"/>
       </geometry>
     </visual>
   </link>
   <link name='wheel_RL'>
-    <xacro:cylinder_inertial name="wheel_RL" m="${wheel_mass}" r="${wheel_radius}" h="${wheel_width}"/>
+    <xacro:cylinder_inertial name="wheel_RL" m="${wheel_mass}" r="${wheel_radius_back}" h="${wheel_width}"/>
     <collision name='wheel_RL_collision'>
       <origin xyz="0 0 0" rpy="1.5708 0 0"/>
       <geometry>
-        <cylinder radius="${wheel_radius}" length="${wheel_width}"/>
+        <cylinder radius="${wheel_radius_back}" length="${wheel_width}"/>
       </geometry>
     </collision>
@@ -87,5 +89,5 @@
       <origin xyz="0 0 0" rpy="1.5708 0 0"/>
       <geometry>
-        <cylinder radius="${wheel_radius}" length="${wheel_width}"/>
+        <cylinder radius="${wheel_radius_back}" length="${wheel_width}"/>
       </geometry>
     </visual>
@@ -108,5 +110,5 @@
     <parent link="chassis"/>
     <child link="wheel_FR"/>
-    <origin xyz="${chassis_length/2-wheel_radius} -${chassis_width/2+wheel_width/2} 0"
+    <origin xyz="${chassis_length/2-wheel_radius_front} -${chassis_width/2+wheel_width/2} 0"
             rpy="0 0 0"/>
     <axis xyz="0 1 0"/>
@@ -115,5 +117,5 @@
     <parent link="chassis"/>
     <child link="wheel_FL"/>
-    <origin xyz="${chassis_length/2-wheel_radius} ${chassis_width/2+wheel_width/2} 0"
+    <origin xyz="${chassis_length/2-wheel_radius_front} ${chassis_width/2+wheel_width/2} 0"
             rpy="0 0 0"/>
     <axis xyz="0 1 0"/>
@@ -122,5 +124,5 @@
     <parent link="chassis"/>
     <child link="wheel_RR"/>
-    <origin xyz="-${chassis_length/2-wheel_radius} -${chassis_width/2+wheel_width/2} 0"
+    <origin xyz="-${chassis_length/2-wheel_radius_back} -${chassis_width/2+wheel_width/2} 0"
             rpy="0 0 0"/>
     <axis xyz="0 1 0"/>
@@ -129,5 +131,5 @@
     <parent link="chassis"/>
     <child link="wheel_RL"/>
-    <origin xyz="-${chassis_length/2-wheel_radius} ${chassis_width/2+wheel_width/2} 0"
+    <origin xyz="-${chassis_length/2-wheel_radius_back} ${chassis_width/2+wheel_width/2} 0"
             rpy="0 0 0"/>
     <axis xyz="0 1 0"/>
@@ -156,3 +158,58 @@
     <material>Gazebo/Yellow</material>
   </gazebo>
+  <gazebo reference="camera_link">
+    <sensor type="camera" name="camera1">
+      <update_rate>30.0</update_rate>
+      <camera name="head">
+        <horizontal_fov>1.3962634</horizontal_fov>
+        <image>
+          <width>600</width>
+          <height>400</height>
+          <format>R8G8B8</format>
+        </image>
+        <clip>
+          <near>0.02</near>
+          <far>300</far>
+        </clip>
+        <noise>
+          <type>gaussian</type>
+          <!-- Noise is sampled independently per pixel on each frame.
+               That pixel's noise value is added to each of its color
+               channels, which at that point lie in the range [0,1]. -->
+          <mean>0.0</mean>
+          <stddev>0.007</stddev>
+        </noise>
+      </camera>
+      <plugin name="camera_controller" filename="libgazebo_ros_camera.so">
+        <alwaysOn>true</alwaysOn>
+        <updateRate>0.0</updateRate>
+        <cameraName>robot/camera1</cameraName>
+        <imageTopicName>image_raw</imageTopicName>
+        <cameraInfoTopicName>camera_info</cameraInfoTopicName>
+        <frameName>camera_link</frameName>
+        <hackBaseline>0.07</hackBaseline>
+        <distortionK1>0.0</distortionK1>
+        <distortionK2>0.0</distortionK2>
+        <distortionK3>0.0</distortionK3>
+        <distortionT1>0.0</distortionT1>
+        <distortionT2>0.0</distortionT2>
+      </plugin>
+    </sensor>
+  </gazebo>
+<gazebo>
+  <plugin name="skid_steer_drive_controller" filename="libgazebo_ros_skid_steer_drive.so">
+    <updateRate>100.0</updateRate>
+    <robotNamespace>/</robotNamespace>
+    <leftFrontJoint>wheel_FL_joint</leftFrontJoint>
+    <rightFrontJoint>wheel_FR_joint</rightFrontJoint>
+    <leftRearJoint>wheel_RL_joint</leftRearJoint>
+    <rightRearJoint>wheel_RR_joint</rightRearJoint>
+    <wheelSeparation>0.4</wheelSeparation>
+    <wheelDiameter>0.215</wheelDiameter>
+    <robotBaseFrame>base_link</robotBaseFrame>
+    <torque>20</torque>
+    <topicName>cmd_vel</topicName>
+    <broadcastTF>false</broadcastTF>
+  </plugin>
+</gazebo>
 </robot>
